File: kicad/Macintosh Portable 50-pin Hard Drive Adapter v1.1.sch (KiCad schematic (older format))
At the start: 4 parts, among them J1 SCSI_SE_Internal_Conn_02x25_O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, J2 Mac_Portable_SCSI_SE_Conn_02x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, J3 171825-4

Commit message: Version 1.1
Parts:
- J1: symbol Connector_Generic_MountingPin:SCSI_SE_Internal_Conn_02x25_Odd_Even_MountingPin -> Macintosh~Portable~50-pin~Hard~Drive~Adapter:SCSI_SE_Internal_Conn_02x25_Odd_Even_MountingPin
- J2: footprint Connector_PinHeader_2.54mm:PinHeader_2x17_P2.54mm_Vertical -> Connector_IDC:IDC-Header_2x17_P2.54mm_Vertical; symbol Connector_Generic_MountingPin:Mac_Portable_SCSI_SE_Conn_02x17_Odd_Even_MountingPin -> Macintosh~Portable~50-pin~Hard~Drive~Adapter:Mac_Portable_SCSI_SE_Conn_02x17_Odd_Even_MountingPin
- J3: symbol mac_portable_34pin_to_50pin_scsi:171825-4 -> snapeda:171825-4
Connections:
- net labels removed: GND1, GND2, GND3, GND4, GNDREF, Ground1, Ground2, Ground3, Ground4
- wire segments 111 -> 148
