File: kicad/Macintosh Portable 50-pin Hard Drive Adapter.kicad_pcb (KiCad board)
At the start: 2 copper layers, 65.5 x 26 mm, 5 parts, among them J1 SCSI_SE_Internal_Conn_02x25_O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, J2 Mac_Portable_SCSI_SE_Conn_02x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, J3 171825-4

Commit message: Version 1.1
Parts:
- J2: footprint Connector_PinHeader_2.54mm:PinHeader_2x17_P2.54mm_Vertical -> Connector_IDC:IDC-Header_2x17_P2.54mm_Vertical
- J3: footprint mac_portable_34pin_to_50pin_scsi:TE_171825-4 -> snapeda:TE_171825-4
